File: MicroFLiC_servo_solenoid_1_0.kicad_pcb (KiCad board)
At the start: 2 copper layers, 49.8 x 49.8 mm, 49 parts, among them P1 Header_1x14, P10 Socket_1x4, P11 Header_R/A_2x3, P12 Header_R/A_2x3, P2 Socket_1x14, P3 12-way Micro-MaTch, P4 Jack_3.5mm_3pin, P5 Jack_3.5mm_3pin, P6 RCA_3, P7 RCA_3, P8 Socket_1x6, P9 Header_1x4, U1 PCA9306, U2 DRV103, U3 DRV103, U4 MCP4728

Commit message: Final production board v1.0
Parts:
- turned D1 to 180 degrees
- turned D2 to 180 degrees
- turned D3 to 180 degrees
- turned D4 to 180 degrees
Connections:
- D1 pad 1: /shutterPWM/EA -> /shutterPWM/ENG_A
- D1 pad 2: /shutterPWM/ENG_A -> /shutterPWM/EA
- D2 pad 1: /shutterPWM/EB -> /shutterPWM/ENG_B
- D2 pad 2: /shutterPWM/ENG_B -> /shutterPWM/EB
- D3 pad 1: /shutterPWM/FA -> /shutterPWM/SHA_O/C
- D3 pad 2: /shutterPWM/SHA_O/C -> /shutterPWM/FA
- D4 pad 1: /shutterPWM/FB -> /shutterPWM/SHB_O/C
- D4 pad 2: /shutterPWM/SHB_O/C -> /shutterPWM/FB
Routing:
- net /shutterPWM/FA: track 0.00 -> 1.69 mm
