File: MicroFLiC_servo_solenoid_1_0.sch (KiCad schematic (older format))
At the start: 14 parts, among them P1 Header_1x14, P10 Socket_1x4, P2 Socket_1x14, P3 12-way Micro-MaTch, P4 Jack_3.5mm_3pin, P5 Jack_3.5mm_3pin, P6 RCA_3, P7 RCA_3, P8 Socket_1x6, P9 Header_1x4

Commit message: Final production board v1.0
Changed lines of the file:
@@
 EESchema Schematic File Version 2
+LIBS:MicroFLiC_servo_solenoid_1_0-rescue
 LIBS:power
 LIBS:device
@@
 $EndComp
 Wire Wire Line
-	2400 6100 2500 6100
+	2300 6100 2500 6100
 Wire Wire Line
 	2500 6100 2500 6300
 Wire Wire Line
-	2500 6300 2400 6300
+	2500 6300 2300 6300
 Connection ~ 2500 6200
 Wire Wire Line
-	1900 6100 1400 6100
-Wire Wire Line
-	1900 6300 1400 6300
-Text Label 1500 6100 0    60   ~ 0
+	2000 6100 1500 6100
+Wire Wire Line
+	2000 6300 1500 6300
+Text Label 1600 6100 0    60   ~ 0
 SERVO1
-Text Label 1500 6300 0    60   ~ 0
+Text Label 1600 6300 0    60   ~ 0
 SERVO3
 Text Label 2600 7100 0    60   ~ 0
@@
 	3000 7000 3000 7200
 Wire Wire Line
-	2400 7000 2500 7000
+	2300 7000 2500 7000
 Wire Wire Line
 	2500 7000 2500 7200
 Wire Wire Line
-	2500 7200 2400 7200
+	2500 7200 2300 7200
 Connection ~ 2500 7100
 Wire Wire Line
-	1900 7000 1400 7000
-Wire Wire Line
-	1900 7200 1400 7200
-Text Label 1500 7000 0    60   ~ 0
+	2000 7000 1500 7000
+Wire Wire Line
+	2000 7200 1500 7200
+Text Label 1600 7000 0    60   ~ 0
 SERVO2
-Text Label 1500 7200 0    60   ~ 0
+Text Label 1600 7200 0    60   ~ 0
 SERVO4
 $Comp

Commit message: Added component descriptions
Parts:
- P1: Manufacturer Samtec -> Multicomp; Order Code 2010798 -> 1593421; Part Number HTSW-114-15-G-S -> MC34735
Changed lines of the file:
@@
 F 2 "Pin_Headers:Pin_Header_Straight_1x14" H 1300 1950 60  0001 C CNN
 F 3 "" H 1300 1950 60  0000 C CNN
-F 4 "HTSW-114-15-G-S" H 1300 1950 60  0001 C CNN "Part Number"
-F 5 "Samtec" H 1300 1950 60  0001 C CNN "Manufacturer"
-F 6 "2010798" H 1300 1950 60  0001 C CNN "Order Code"
+F 4 "MC34735" H 1300 1950 60  0001 C CNN "Part Number"
+F 5 "Multicomp" H 1300 1950 60  0001 C CNN "Manufacturer"
+F 6 "1593421" H 1300 1950 60  0001 C CNN "Order Code"
 	1    1300 1950
 	-1   0    0    -1
